File: ETL.kicad_pcb (KiCad board)
At the start: 2 copper layers, 10 x 12 mm, 16 parts, among them U1 SolderPad, U10 SolderPad, U11 SolderPad, U13 SolderPad, U15 SolderPad, U4 SolderPad, U6 SolderPad, U8 SolderPad

Commit message: i am updating the pcb
Parts:
- U1, U11, U4, U8: moved to F.Cu
- moved U11 4.59 mm to (182.5, 118.5)
- moved U4 4.59 mm to (180.0, 118.5)
- moved U1 4.54 mm to (175.0, 118.5)
- moved U10 4.36 mm to (177.5, 115.0)
- moved U13 4.31 mm to (180.0, 115.0)
- moved U6 4.31 mm to (182.5, 115.0)
- moved U8 4.12 mm to (177.5, 118.5)
- moved U11 4.00 mm to (182.5, 120.8)
- moved U6 4.00 mm to (182.5, 120.8)
- moved U1 3.96 mm to (175.0, 120.8)
- moved U15 3.94 mm to (175.0, 120.8)
- moved U13 3.93 mm to (180.0, 120.8)
- moved U4 3.93 mm to (180.0, 120.8)
- moved U10 3.92 mm to (177.5, 120.8)
- moved U8 3.92 mm to (177.5, 120.8)
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Other:
- outline, holes or cut-outs redrawn
